File: kicad/PowerSource.kicad_sch (KiCad schematic)
At the start: 30 parts, among them U13 AMS1117-3.3, U3 MP9488GS-Z, U5 AP63205

Commit message: made full cell balancing up to 36S
Other:
- note added: "7.5V-450V to 15V"
- note removed: "Battery voltage to 15V"
Changed lines of the file:
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@@
     (effects (font (size 1.27 1.27)) (justify left bottom))
   )
-  (text "Battery voltage to 15V" (at 58.42 52.07 0)
+  (text "7.5V-450V to 15V" (at 58.42 52.07 0)
     (effects (font (size 1.27 1.27)) (justify left bottom))
   )
