File: kicad/CellTempMonitor.kicad_sch (KiCad schematic)
At the start: 2 parts, among them U60 LTC4318, U61 MLX90632

Commit message: Added MLX90632 IR temperature sensor
Parts:
- removed U60: LTC4318, Package_DFN_QFN:QFN-20-1EP_4x4mm_P0.5mm_EP2.5x2.5mm, symbol sBMS:LTC4318
- removed U61: MLX90632, symbol sBMS:MLX90632
Changed lines of the file:
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@@
 (kicad_sch (version 20230121) (generator eeschema)
   (paper "A4")
-  (symbol (lib_id "sBMS:LTC4318") (at 143.51 93.98 0) (unit 1)
-    (in_bom yes) (on_board yes) (dnp no) (fields_autoplaced)
-    (property "Reference" "U60" (at 145.7041 71.12 0)
-      (effects (font (size 1.27 1.27)) (justify left))
-    )
-    (property "Value" "LTC4318" (at 145.7041 73.66 0)
-      (effects (font (size 1.27 1.27)) (justify left))
-    )
-    (property "Footprint" "Package_DFN_QFN:QFN-20-1EP_4x4mm_P0.5mm_EP2.5x2.5mm" (at 143.51 118.11 0)
-      (effects (font (size 1.27 1.27)) hide)
-    )
-    (property "Datasheet" "" (at 143.51 88.9 0)
-      (effects (font (size 1.27 1.27)) hide)
-    )
-    (pin "1")
-    (pin "10")
-    (pin "11")
-    (pin "12")
-    (pin "13")
-    (pin "14")
-    (pin "15")
-    (pin "16")
-    (pin "17")
-    (pin "19")
-    (pin "2")
-    (pin "20")
-    (pin "21")
-    (pin "3")
-    (pin "4")
-    (pin "5")
-    (pin "6")
-    (pin "7")
-    (pin "8")
-    (instances
-      (project "sBMS"
-        (path "/7f25f26f-13d1-483f-a85d-b3abae309e30/12d9a724-445f-445b-89ea-1a4697ea3bb2/868a2eef-58b0-48b8-ace3-d30f6b0d6274"
-          (reference "U60") (unit 1)
-        )
-      )
-    )
-  )
-  (symbol (lib_id "sBMS:MLX90632") (at 101.6 128.27 0) (unit 1)
-    (in_bom yes) (on_board yes) (dnp no) (fields_autoplaced)
-    (property "Reference" "U61" (at 114.3 124.6221 0)
-      (effects (font (size 1.27 1.27)))
-    )
-    (property "Value" "MLX90632" (at 114.3 127.1621 0)
-      (effects (font (size 1.27 1.27)))
-    )
-    (property "Footprint" "" (at 101.6 128.27 0)
-      (effects (font (size 1.27 1.27)) hide)
-    )
-    (property "Datasheet" "" (at 101.6 128.27 0)
-      (effects (font (size 1.27 1.27)) hide)
-    )
-    (pin "1")
-    (pin "2")
-    (pin "3")
-    (pin "4")
-    (pin "5")
-    (instances
-      (project "sBMS"
-        (path "/7f25f26f-13d1-483f-a85d-b3abae309e30/12d9a724-445f-445b-89ea-1a4697ea3bb2/868a2eef-58b0-48b8-ace3-d30f6b0d6274"
-          (reference "U61") (unit 1)
-        )
-      )
-    )
-  )
 )

Commit message: removed center mounted humidity sensors (HDC302x)
Parts:
- added U60: LTC4318, Package_DFN_QFN:QFN-20-1EP_4x4mm_P0.5mm_EP2.5x2.5mm, symbol sBMS:LTC4318
- added U61: MLX90632, symbol sBMS:MLX90632
Changed lines of the file:
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@@
 (kicad_sch (version 20230121) (generator eeschema)
   (paper "A4")
+  (symbol (lib_id "sBMS:LTC4318") (at 143.51 93.98 0) (unit 1)
+    (in_bom yes) (on_board yes) (dnp no) (fields_autoplaced)
+    (property "Reference" "U60" (at 145.7041 71.12 0)
+      (effects (font (size 1.27 1.27)) (justify left))
+    )
+    (property "Value" "LTC4318" (at 145.7041 73.66 0)
+      (effects (font (size 1.27 1.27)) (justify left))
+    )
+    (property "Footprint" "Package_DFN_QFN:QFN-20-1EP_4x4mm_P0.5mm_EP2.5x2.5mm" (at 143.51 118.11 0)
+      (effects (font (size 1.27 1.27)) hide)
+    )
+    (property "Datasheet" "" (at 143.51 88.9 0)
+      (effects (font (size 1.27 1.27)) hide)
+    )
+    (pin "1")
+    (pin "10")
+    (pin "11")
+    (pin "12")
+    (pin "13")
+    (pin "14")
+    (pin "15")
+    (pin "16")
+    (pin "17")
+    (pin "19")
+    (pin "2")
+    (pin "20")
+    (pin "21")
+    (pin "3")
+    (pin "4")
+    (pin "5")
+    (pin "6")
+    (pin "7")
+    (pin "8")
+    (instances
+      (project "sBMS"
+        (path "/7f25f26f-13d1-483f-a85d-b3abae309e30/12d9a724-445f-445b-89ea-1a4697ea3bb2/868a2eef-58b0-48b8-ace3-d30f6b0d6274"
+          (reference "U60") (unit 1)
+        )
+      )
+    )
+  )
+  (symbol (lib_id "sBMS:MLX90632") (at 101.6 128.27 0) (unit 1)
+    (in_bom yes) (on_board yes) (dnp no) (fields_autoplaced)
+    (property "Reference" "U61" (at 114.3 124.6221 0)
+      (effects (font (size 1.27 1.27)))
+    )
+    (property "Value" "MLX90632" (at 114.3 127.1621 0)
+      (effects (font (size 1.27 1.27)))
+    )
+    (property "Footprint" "" (at 101.6 128.27 0)
+      (effects (font (size 1.27 1.27)) hide)
+    )
+    (property "Datasheet" "" (at 101.6 128.27 0)
+      (effects (font (size 1.27 1.27)) hide)
+    )
+    (pin "1")
+    (pin "2")
+    (pin "3")
+    (pin "4")
+    (pin "5")
+    (instances
+      (project "sBMS"
+        (path "/7f25f26f-13d1-483f-a85d-b3abae309e30/12d9a724-445f-445b-89ea-1a4697ea3bb2/868a2eef-58b0-48b8-ace3-d30f6b0d6274"
+          (reference "U61") (unit 1)
+        )
+      )
+    )
+  )
 )
