File: kicad/CellMonitoring.kicad_sch (KiCad schematic)
At the start: 57 parts, among them J7 Conn_01x04, U1 HDC3022, U11 TMCS1123x3, U12 DAC7571, U13 DAC7571, U14 TMCS1123x3, U17 LTC6803-4, U20 LTC6803-4, U21 LTC6803-4, U3 HDC3022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

Commit message: Small refactors
Other:
- moved on the sheet: R2, R3
Changed lines of the file:
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@@
     (stroke (width 0) (type default))
   )
-  (wire (pts (xy 254 26.67) (xy 256.54 26.67))
+  (wire (pts (xy 252.73 43.18) (xy 255.27 43.18))
     (stroke (width 0) (type default))
   )
@@
     )
   )
-  (global_label "Bat_Voltage" (shape input) (at 255.27 26.67 270) (fields_autoplaced)
+  (global_label "Bat_Voltage" (shape input) (at 254 43.18 270) (fields_autoplaced)
     (effects (font (size 1.27 1.27)) (justify right))
-    (property "Intersheetrefs" "${INTERSHEET_REFS}" (at 255.27 40.7826 90)
+    (property "Intersheetrefs" "${INTERSHEET_REFS}" (at 254 57.2926 90)
       (effects (font (size 1.27 1.27)) (justify right) hide)
     )
@@
     )
   )
-  (symbol (lib_id "Device:R") (at 260.35 26.67 90) (unit 1)
-    (in_bom yes) (on_board yes) (dnp no) (fields_autoplaced)
-    (property "Reference" "R3" (at 260.35 20.32 90)
-      (effects (font (size 1.27 1.27)))
-    )
-    (property "Value" "50k" (at 260.35 22.86 90)
-      (effects (font (size 1.27 1.27)))
-    )
-    (property "Footprint" "" (at 260.35 28.448 90)
-      (effects (font (size 1.27 1.27)) hide)
-    )
-    (property "Datasheet" "~" (at 260.35 26.67 0)
+  (symbol (lib_id "Device:R") (at 259.08 43.18 90) (unit 1)
+    (in_bom yes) (on_board yes) (dnp no) (fields_autoplaced)
+    (property "Reference" "R3" (at 259.08 36.83 90)
+      (effects (font (size 1.27 1.27)))
+    )
+    (property "Value" "50k" (at 259.08 39.37 90)
+      (effects (font (size 1.27 1.27)))
+    )
+    (property "Footprint" "" (at 259.08 44.958 90)
+      (effects (font (size 1.27 1.27)) hide)
+    )
+    (property "Datasheet" "~" (at 259.08 43.18 0)
       (effects (font (size 1.27 1.27)) hide)
     )
@@
     )
   )
-  (symbol (lib_id "power:+BATT") (at 264.16 26.67 270) (unit 1)
-    (in_bom yes) (on_board yes) (dnp no) (fields_autoplaced)
-    (property "Reference" "#PWR011" (at 260.35 26.67 0)
-      (effects (font (size 1.27 1.27)) hide)
-    )
-    (property "Value" "+BATT" (at 267.97 26.67 90)
+  (symbol (lib_id "power:+BATT") (at 262.89 43.18 270) (unit 1)
+    (in_bom yes) (on_board yes) (dnp no) (fields_autoplaced)
+    (property "Reference" "#PWR011" (at 259.08 43.18 0)
+      (effects (font (size 1.27 1.27)) hide)
+    )
+    (property "Value" "+BATT" (at 266.7 43.18 90)
       (effects (font (size 1.27 1.27)) (justify left))
     )
-    (property "Footprint" "" (at 264.16 26.67 0)
-      (effects (font (size 1.27 1.27)) hide)
-    )
-    (property "Datasheet" "" (at 264.16 26.67 0)
+    (property "Footprint" "" (at 262.89 43.18 0)
+      (effects (font (size 1.27 1.27)) hide)
+    )
+    (property "Datasheet" "" (at 262.89 43.18 0)
       (effects (font (size 1.27 1.27)) hide)
     )
@@
     )
   )
-  (symbol (lib_id "power:GND") (at 246.38 26.67 270) (unit 1)
-    (in_bom yes) (on_board yes) (dnp no) (fields_autoplaced)
-    (property "Reference" "#PWR010" (at 240.03 26.67 0)
-      (effects (font (size 1.27 1.27)) hide)
-    )
-    (property "Value" "GND" (at 242.57 26.67 90)
+  (symbol (lib_id "power:GND") (at 245.11 43.18 270) (unit 1)
+    (in_bom yes) (on_board yes) (dnp no) (fields_autoplaced)
+    (property "Reference" "#PWR010" (at 238.76 43.18 0)
+      (effects (font (size 1.27 1.27)) hide)
+    )
+    (property "Value" "GND" (at 241.3 43.18 90)
       (effects (font (size 1.27 1.27)) (justify right))
     )
-    (property "Footprint" "" (at 246.38 26.67 0)
-      (effects (font (size 1.27 1.27)) hide)
-    )
-    (property "Datasheet" "" (at 246.38 26.67 0)
+    (property "Footprint" "" (at 245.11 43.18 0)
+      (effects (font (size 1.27 1.27)) hide)
+    )
+    (property "Datasheet" "" (at 245.11 43.18 0)
       (effects (font (size 1.27 1.27)) hide)
     )
@@
     )
   )
-  (symbol (lib_id "Device:R") (at 250.19 26.67 90) (unit 1)
-    (in_bom yes) (on_board yes) (dnp no) (fields_autoplaced)
-    (property "Reference" "R2" (at 250.19 20.32 90)
-      (effects (font (size 1.27 1.27)))
-    )
-    (property "Value" "1k" (at 250.19 22.86 90)
-      (effects (font (size 1.27 1.27)))
-    )
-    (property "Footprint" "" (at 250.19 28.448 90)
-      (effects (font (size 1.27 1.27)) hide)
-    )
-    (property "Datasheet" "~" (at 250.19 26.67 0)
-      (effects (font (size 1.27 1.27)) hide)
-    )
+  (symbol (lib_id "Device:R") (at 248.92 43.18 90) (unit 1)
+    (in_bom yes) (on_board yes) (dnp no) (fields_autoplaced)
+    (property "Reference" "R2" (at 248.92 36.83 90)
+      (effects (font (size 1.27 1.27)))
+    )
+    (property "Value" "1k" (at 248.92 39.37 90)
+      (effects (font (size 1.27 1.27)))
+    )
+    (property "Footprint" "" (at 248.92 44.958 90)
+      (effects (font (size 1.27 1.27)) hide)
+    )
+    (property "Datasheet" "~" (at 248.92 43.18 0)
+      (effects (font (size 1.27 1.27)) hide)
+    )

Commit message: More refactors for the god of refactors
Parts:
- removed U3, U4, U5, U6: HDC3022, Package_SON:Texas_S-PWSON-N8_EP1.2x2mm, symbol Sensor_Humidity:HDC3022
Other:
- note added: "This circuit can be repeated multiple times. It's designed to be used with a separate "programmer" device that programms the I2C address inside the sensors's EEPROM, and connects via the connector on the left."
- note added: "You can change ADDR and ADDR1 connections to ground and +5V to make this IC have different I2C addresses, if you repeat this circuit multiple times"
- note removed: "Bottom left"
- note removed: "Bottom right"
- note removed: "Charge FET"
- note removed: "This circuit can be repeated multiple times. It's designed to be used with a separate "programmer" device that programms the I2C address inside the sensors's EEPROM."
- note removed: "Top left"
- note removed: "Top right"
- moved on the sheet: C3, C4, J7, JP1, R80, R81, U1, U11, U12, U13, U14, U61
