File: kicad/CellMonitoring.kicad_sch (KiCad schematic)
At the start: 53 parts, among them J7 Conn_01x04, U1 HDC3022, U11 TMCS1123x3, U12 DAC7571, U13 DAC7571, U14 TMCS1123x3, U17 LTC6803-4, U20 LTC6803-4, U21 LTC6803-4, U61 MLX90632

Commit message: Finished SBMS-T-3, started work on SBMS-T-4
Parts:
- renumbered R81 to R80, R80 to R81, U61 to U7
Changed lines of the file:
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@@
   (symbol (lib_id "power:+5V") (at 90.17 110.49 0) (unit 1)
     (in_bom yes) (on_board yes) (dnp no) (fields_autoplaced)
-    (property "Reference" "#PWR034" (at 90.17 114.3 0)
+    (property "Reference" "#PWR035" (at 90.17 114.3 0)
       (effects (font (size 1.27 1.27)) hide)
     )
@@
   (symbol (lib_id "power:GND") (at 72.39 133.35 0) (unit 1)
     (in_bom yes) (on_board yes) (dnp no) (fields_autoplaced)
-    (property "Reference" "#PWR036" (at 72.39 139.7 0)
+    (property "Reference" "#PWR034" (at 72.39 139.7 0)
       (effects (font (size 1.27 1.27)) hide)
     )
@@
   (symbol (lib_id "Device:R") (at 81.28 121.92 0) (mirror y) (unit 1)
     (in_bom yes) (on_board yes) (dnp no)
-    (property "Reference" "R80" (at 82.55 119.38 0)
+    (property "Reference" "R81" (at 82.55 119.38 0)
       (effects (font (size 1.27 1.27)) (justify right))
     )
@@
   (symbol (lib_id "Device:R") (at 74.93 123.19 0) (mirror y) (unit 1)
     (in_bom yes) (on_board yes) (dnp no)
-    (property "Reference" "R81" (at 76.2 120.65 0)
+    (property "Reference" "R80" (at 76.2 120.65 0)
       (effects (font (size 1.27 1.27)) (justify right))
     )
@@
   (symbol (lib_id "power:GND") (at 90.17 138.43 0) (unit 1)
     (in_bom yes) (on_board yes) (dnp no) (fields_autoplaced)
-    (property "Reference" "#PWR035" (at 90.17 144.78 0)
+    (property "Reference" "#PWR036" (at 90.17 144.78 0)
       (effects (font (size 1.27 1.27)) hide)
     )
@@
   (symbol (lib_id "sBMS:MLX90632") (at 90.17 129.54 0) (unit 1)
     (in_bom yes) (on_board yes) (dnp no)
-    (property "Reference" "U61" (at 97.79 121.92 0)
+    (property "Reference" "U7" (at 97.79 121.92 0)
       (effects (font (size 1.27 1.27)) (justify left))
     )
